Commit message: added robot visual urdf need to add c0ollison and inertial prop

File: benzene_description/urdf/mech/base.urdf.xacro (robot description, xacro)
@@ -1,56 +1,73 @@
 <?xml version="1.0"?>
 <robot xmlns:xacro="http://www.ros.org/wiki/xacro">
-<xacro:property name="total_width" value="0.19940" />
-<xacro:property name="wheel_width" value="0.0304" />
-<xacro:property name="wheel_radius" value="0.0325" />
-<xacro:property name="total_height" value="0.26225" />
-<xacro:property name="base_length" value="0.300" />
-<xacro:property name="centered_length" value="0.238" />
-<xacro:property name="base_x_offset" value="${(centered_length - base_length) / 2}" />
-<xacro:property name="base_size_x" value="${base_length}" />
-<xacro:property name="base_size_y" value="${total_width - (2 * wheel_width)}" />
-<xacro:property name="base_size_z" value="${total_height - (2 * wheel_radius)}" />
-<xacro:property name="base_mass" value="4.6" />
-<xacro:macro name="rosmaster_x3_base" params="prefix">
-  <link name="${prefix}base_footprint"/>
-  <link name="${prefix}base_link">
-    <visual>
+  <!-- =========================
+       BASE DIMENSIONS
+       ========================= -->
+  <xacro:property name="base_length" value="0.300"/>
+  <xacro:property name="base_width" value="0.19940"/>
+  <xacro:property name="base_height" value="0.040"/>
+  <xacro:property name="base_mass" value="4.6"/>
+  <!-- =========================
+       BASE MACRO
+       ========================= -->
+  <xacro:macro name="base" params="prefix">
+    <!-- BASE FOOTPRINT -->
+    <link name="${prefix}base_footprint"/>
+    <!-- BASE LINK -->
+    <link name="${prefix}base_link">
+      <visual>
+        <origin xyz="0 0 0" rpy="0 0 0"/>
         <geometry>
-            <mesh filename="file://$(find benzene_description)/meshes/benzene/visual/chassis.stl"/>
+          <mesh
+            filename="file://$(find benzene_description)/meshes/benzene/visual/chassis.stl"
+            scale="0.001 0.001 0.001"/>
         </geometry>
         <material name="green">
           <color rgba="0 0.7 0 1"/>
         </material>
-        <origin xyz="0 0 0" rpy="0 0 0"/>
-    </visual>
-    <collision>
+      </visual>
+      <collision>
         <geometry>
-            <box size="${base_size_x} ${base_size_y} ${base_size_z}"/>
+          <box
+            size="${base_length} ${base_width} ${base_height}"/>
         </geometry>
-        <origin xyz="${base_x_offset} 0 ${base_size_z/2 + wheel_radius/4}" rpy="0 0 0"/>
-    </collision>
-    <inertial>
-        <origin xyz="${base_x_offset} 0 ${base_size_z/2 + wheel_radius/4}" rpy="0 0 0"/>
+        <origin
+          xyz="0 0 0"
+          rpy="0 0 0"/>
+      </collision>
+      <inertial>
+        <origin
+          xyz="0 0 0"
+          rpy="0 0 0"/>
         <mass value="${base_mass}"/>
         <inertia
-            ixx="${(1/12) * base_mass * ((base_size_y * base_size_y) + (base_size_z * base_size_z))}" ixy="0.0" ixz="0.0"
-            iyy="${(1/12) * base_mass * ((base_size_x * base_size_x) + (base_size_z * base_size_z))}" iyz="0.0"
-            izz="${(1/12) * base_mass * ((base_size_x * base_size_x) + (base_size_y * base_size_y))}"/>
-    </inertial>
-  </link>
-  <gazebo reference="${prefix}base_link">
-    <visual>
+          ixx="${(1/12) * base_mass * (base_width*base_width + base_height*base_height)}"
+          ixy="0"
+          ixz="0"
+          iyy="${(1/12) * base_mass * (base_length*base_length + base_height*base_height)}"
+          iyz="0"
+          izz="${(1/12) * base_mass * (base_length*base_length + base_width*base_width)}"/>
+      </inertial>
+    </link>
+    <!-- BASE FOOTPRINT -> BASE LINK -->
+    <joint
+      name="${prefix}base_footprint_joint"
+      type="fixed">
+      <parent link="${prefix}base_footprint"/>
+      <child link="${prefix}base_link"/>
+      <origin
+        xyz="0 0 0"
+        rpy="0 0 0"/>
+    </joint>
+    <!-- GAZEBO MATERIAL -->
+    <gazebo reference="${prefix}base_link">
+      <visual>
         <material>
-            <ambient>0 0.7 0 1</ambient>
-            <diffuse>0 0.7 0 1</diffuse>
-            <specular>0 0.7 0 1</specular>
+          <ambient>0 0.7 0 1</ambient>
+          <diffuse>0 0.7 0 1</diffuse>
+          <specular>0 0.7 0 1</specular>
         </material>
-    </visual>
-  </gazebo>
-  <joint name="${prefix}base_joint" type="fixed">
-    <parent link="${prefix}base_footprint"/>
-    <child link="${prefix}base_link"/>
-    <origin xyz="0 0 ${wheel_radius}" rpy="0 0 0"/>
-  </joint>
-</xacro:macro>
+      </visual>
+    </gazebo>
+  </xacro:macro>
 </robot>

File: benzene_description/urdf/mech/wheel.urdf.xacro (robot description, xacro)
@@ -1,60 +1,119 @@
 <?xml version="1.0"?>
 <robot xmlns:xacro="http://www.ros.org/wiki/xacro">
-  <xacro:property name="wheel_radius" value="0.035" />
-  <xacro:property name="wheel_separation" value="0.207" />
-  <xacro:property name="wheel_width" value="0.02666" />
-  <xacro:property name="wheel_mass" value="9.1" />
-  <xacro:property name="wheel_xoff" value="0.08" />
-  <xacro:property name="wheel_yoff" value="-0.01" />
-  <xacro:macro name="wheel" params="prefix side x_reflect y_reflect">
-    <link name="${prefix}${side}_wheel_link">
-      <visual>
-        <origin xyz="0 0 0" rpy="${pi/2} 0 0"/>
-        <geometry>
-          <mesh filename="file://$(find benzene_description)/meshes/benzene/visual/${side}_wheel.stl"/>
-        </geometry>
-        <material name="dark_gray">
-          <color rgba="0.2 0.2 0.2 1.0"/>
-        </material>
-      </visual>
-      <collision>
-        <origin xyz="0 0 0" rpy="${pi/2} 0 0"/>
-        <geometry>
-          <cylinder radius="${wheel_radius}" length="${wheel_width}"/>
-        </geometry>
-      </collision>
-      <inertial>
-        <origin xyz="0 0 0" rpy="0 0 0"/>
-        <mass value="${wheel_mass}"/>
-        <inertia
-          ixx="${(wheel_mass/12.0) * (3*wheel_radius*wheel_radius + wheel_width*wheel_width)}" ixy="0" ixz="0"
-          iyy="${(wheel_mass/2.0) * (wheel_radius*wheel_radius)}" iyz="0"
-          izz="${(wheel_mass/12.0) * (3*wheel_radius*wheel_radius + wheel_width*wheel_width)}"/>
-      </inertial>
-    </link>
-    <joint name="${prefix}${side}_wheel_joint" type="continuous">
-      <axis xyz="0 1 0"/>
-      <parent link="${prefix}base_link"/>
-      <child link="${prefix}${side}_wheel_link"/>
-      <origin xyz="${x_reflect*wheel_xoff} ${y_reflect*(wheel_separation/2+wheel_yoff)} ${-wheel_radius}" rpy="0 0 0"/>
-    </joint>
-    <gazebo reference="${prefix}${side}_wheel_link">
-      <surface>
-        <friction>
-          <ode>
-              <mu>1.0</mu>
-              <mu2>0.0</mu2>
-          </ode>
-        </friction>
-      </surface>
-      <visual>
-          <material>
-              <ambient>0.2 0.2 0.2 1.0</ambient>
-              <diffuse>0.2 0.2 0.2 1.0</diffuse>
-              <specular>0.2 0.2 0.2 1.0</specular>
-              <emissive>0.0 0.0 0.0 0.0</emissive>
-          </material>
-      </visual>
-  </gazebo>
-  </xacro:macro>
+    <!-- =========================================================
+         WHEEL PARAMETERS
+         ========================================================= -->
+    <!-- Wheel physical dimensions -->
+    <xacro:property name="wheel_radius" value="0.035"/>
+    <xacro:property name="wheel_width" value="0.020"/>
+    <!-- Distance between left and right wheel centers -->
+    <xacro:property name="wheel_separation" value="0.180"/>
+    <!-- Wheel position relative to base_link -->
+    <xacro:property name="wheel_x_offset" value="0.0"/>
+    <xacro:property name="wheel_z_offset" value="0.020"/>
+    <!-- Wheel mass -->
+    <xacro:property name="wheel_mass" value="0.2"/>
+    <!-- =========================================================
+         WHEEL MACRO
+         ========================================================= -->
+    <xacro:macro name="wheel"
+                 params="prefix side x_reflect y_reflect">
+        <!-- =====================================================
+             LEFT / RIGHT WHEEL LINK
+             ===================================================== -->
+        <link name="${prefix}${side}_wheel_link">
+            <!-- =================================================
+                 VISUAL
+                 ================================================= -->
+            <visual>
+                <origin
+                    xyz="0 0 0"
+                    rpy="${-y_reflect * pi/2} 0 0"/>
+                <geometry>
+                    <mesh
+                        filename="file://$(find benzene_description)/meshes/benzene/visual/${side}_wheel.stl"
+                        scale="0.001 0.001 0.001"/>
+                </geometry>
+                <material name="blue">
+                    <color rgba="0 0 1 1"/>
+                </material>
+            </visual>
+            <!-- =================================================
+                 COLLISION
+                 ================================================= -->
+            <collision>
+                <origin
+                    xyz="0 0 0"
+                    rpy="0 0 0"/>
+                <geometry>
+                    <cylinder
+                        radius="${wheel_radius}"
+                        length="${wheel_width}"/>
+                </geometry>
+            </collision>
+            <!-- =================================================
+                 INERTIAL
+                 ================================================= -->
+            <inertial>
+                <origin
+                    xyz="0 0 0"
+                    rpy="0 0 0"/>
+                <mass value="${wheel_mass}"/>
+                <inertia
+                    ixx="${(wheel_mass / 12.0) * (3.0 * wheel_radius * wheel_radius + wheel_width * wheel_width)}"
+                    ixy="0.0"
+                    ixz="0.0"
+                    iyy="${(wheel_mass / 2.0) * wheel_radius * wheel_radius}"
+                    iyz="0.0"
+                    izz="${(wheel_mass / 12.0) * (3.0 * wheel_radius * wheel_radius + wheel_width * wheel_width)}"/>
+            </inertial>
+        </link>
+        <!-- =====================================================
+             LEFT / RIGHT WHEEL JOINT
+             ===================================================== -->
+        <joint
+            name="${prefix}${side}_wheel_joint"
+            type="continuous">
+            <parent link="${prefix}base_link"/>
+            <child link="${prefix}${side}_wheel_link"/>
+            <!--
+                LEFT:
+                    X = 0
+                    Y = +0.09
+                    Z = +0.02
+                RIGHT:
+                    X = 0
+                    Y = -0.09
+                    Z = +0.02
+            -->
+            <origin
+                xyz="${x_reflect * wheel_x_offset}
+                      ${y_reflect * (wheel_separation / 2.0)}
+                      ${wheel_z_offset}"
+                rpy="0 0 0"/>
+            <!-- Same wheel rotation axis as the original model -->
+            <axis xyz="0 1 0"/>
+        </joint>
+        <!-- =====================================================
+             GAZEBO PARAMETERS
+             ===================================================== -->
+        <gazebo reference="${prefix}${side}_wheel_link">
+            <surface>
+                <friction>
+                    <ode>
+                        <mu>1.0</mu>
+                        <mu2>1.0</mu2>
+                    </ode>
+                </friction>
+            </surface>
+            <visual>
+                <material>
+                    <ambient>0 0 1 1</ambient>
+                    <diffuse>0 0 1 1</diffuse>
+                    <specular>0 0 1 1</specular>
+                    <emissive>0 0 0 0</emissive>
+                </material>
+            </visual>
+        </gazebo>
+    </xacro:macro>
 </robot>

File: benzene_description/urdf/robots/benzene.urdf.xacro (robot description, xacro)
@@ -1,40 +1,216 @@
 <?xml version="1.0"?>
-<robot xmlns:xacro="http://www.ros.org/wiki/xacro" name="rosmaster_x3">
-    <xacro:property name="M_PI" value="3.1415926535897931" />
-    <xacro:arg name="robot_name" default="benzene"/>
-    <xacro:arg name="prefix" default=""/>
-    <xacro:arg name="use_gazebo" default="false"/>
-    <xacro:include filename="$(find benzene_description)/urdf/mech/base.urdf.xacro"/>
-    <xacro:include filename="$(find benzene_description)/urdf/mech/wheel.urdf.xacro"/>
-    <!-- <xacro:include filename="$(find benzene_description)/urdf/sensors/rgbd_camera.urdf.xacro"/> -->
-    <xacro:include filename="$(find benzene_description)/urdf/sensors/lidar.urdf.xacro"/>
-    <xacro:include filename="$(find benzene_description)/urdf/sensors/imu.urdf.xacro"/>
-    <xacro:base prefix="$(arg prefix)"/>
-    <xacro:wheel
-      prefix="$(arg prefix)"
-      side="left"
-      x_reflect="1"
-      y_reflect="1"/>
-    <xacro:wheel
-      prefix="$(arg prefix)"
-      side="right"
-      x_reflect="1"
-      y_reflect="-1"/>
-    <xacro:lidar_sensor
-      prefix="$(arg prefix)"
-      parent="base_link"
-      frame_id="laser_frame"
-      xyz_offset="0 0 0.0825"
-      rpy_offset="0 0 0"
-      mesh_xyz_offset="0 0 0"
-      mesh_rpy_offset="${-M_PI/2} 0 0"
-      topic_name="scan"/>
-    <xacro:imu_sensor
-      prefix="$(arg prefix)"
-      parent="base_link"
-      frame_id="imu"
-      xyz_offset="0 0 0.006"
-      rpy_offset="0 0 0"
-      update_rate="15.0"
-      topic_name="imu/data"/>
+<robot
+  xmlns:xacro="http://www.ros.org/wiki/xacro"
+  name="benzene">
+  <!-- =========================================================
+       CONSTANTS
+       ========================================================= -->
+  <xacro:property
+    name="M_PI"
+    value="3.1415926535897931"/>
+  <!-- =========================================================
+       ARGUMENTS
+       ========================================================= -->
+  <xacro:arg
+    name="robot_name"
+    default="benzene"/>
+  <xacro:arg
+    name="prefix"
+    default=""/>
+  <xacro:arg
+    name="use_gazebo"
+    default="false"/>
+  <!-- =========================================================
+       MECHANICAL COMPONENTS
+       ========================================================= -->
+  <xacro:include
+    filename="$(find benzene_description)/urdf/mech/base.urdf.xacro"/>
+  <xacro:include
+    filename="$(find benzene_description)/urdf/mech/wheel.urdf.xacro"/>
+  <!-- =========================================================
+       SENSORS
+       ========================================================= -->
+  <!-- Camera disabled for now -->
+  <!--
+  <xacro:include
+    filename="$(find benzene_description)/urdf/sensors/camera.urdf.xacro"/>
+  -->
+  <xacro:include
+    filename="$(find benzene_description)/urdf/sensors/lidar.urdf.xacro"/>
+  <xacro:include
+    filename="$(find benzene_description)/urdf/sensors/imu.urdf.xacro"/>
+  <!-- =========================================================
+       BASE
+       ========================================================= -->
+  <xacro:base
+    prefix="$(arg prefix)"/>
+  <!-- =========================================================
+       LEFT DRIVE WHEEL
+       ========================================================= -->
+  <xacro:wheel
+    prefix="$(arg prefix)"
+    side="left"
+    x_reflect="1"
+    y_reflect="1"/>
+  <!-- =========================================================
+       RIGHT DRIVE WHEEL
+       ========================================================= -->
+  <xacro:wheel
+    prefix="$(arg prefix)"
+    side="right"
+    x_reflect="1"
+    y_reflect="-1"/>
+  <!-- =========================================================
+       LIDAR
+       ========================================================= -->
+  <xacro:lidar_sensor
+    prefix="$(arg prefix)"
+    parent="base_link"
+    frame_id="laser_frame"
+    xyz_offset="-0.06 0 0.096"
+    rpy_offset="0 0 0"
+    mesh_xyz_offset="0 0 0"
+    mesh_rpy_offset="0 0 0"
+    topic_name="scan"/>
+  <!-- =========================================================
+       IMU
+       ========================================================= -->
+  <xacro:imu_sensor
+    prefix="$(arg prefix)"
+    parent="base_link"
+    frame_id="imu"
+    xyz_offset="0 0 0.006"
+    rpy_offset="0 0 0"
+    update_rate="15.0"
+    topic_name="imu/data"/>
+  <!-- =========================================================
+       FRONT CASTER WHEEL
+       ========================================================= -->
+  <joint
+    name="$(arg prefix)front_caster_wheel_joint"
+    type="fixed">
+    <parent link="$(arg prefix)base_link"/>
+    <child link="$(arg prefix)front_caster_wheel"/>
+    <!-- Same position as original articubot_two -->
+    <origin
+      xyz="0.12 0 0"
+      rpy="0 0 0"/>
+  </joint>
+  <link name="$(arg prefix)front_caster_wheel">
+    <!-- VISUAL -->
+    <visual>
+      <origin
+        xyz="0 0 0"
+        rpy="0 0 0"/>
+      <geometry>
+        <sphere
+          radius="0.01495"/>
+      </geometry>
+      <material name="caster_black">
+        <color
+          rgba="0 0 0 1"/>
+      </material>
+    </visual>
+    <!-- COLLISION -->
+    <collision>
+      <origin
+        xyz="0 0 0"
+        rpy="0 0 0"/>
+      <geometry>
+        <sphere
+          radius="0.01495"/>
+      </geometry>
+    </collision>
+    <!-- INERTIAL -->
+    <inertial>
+      <origin
+        xyz="0 0 0"
+        rpy="0 0 0"/>
+      <mass
+        value="0.1"/>
+      <inertia
+        ixx="${(2.0/5.0) * 0.1 * 0.01495 * 0.01495}"
+        ixy="0"
+        ixz="0"
+        iyy="${(2.0/5.0) * 0.1 * 0.01495 * 0.01495}"
+        iyz="0"
+        izz="${(2.0/5.0) * 0.1 * 0.01495 * 0.01495}"/>
+    </inertial>
+  </link>
+  <!-- GAZEBO -->
+  <gazebo
+    reference="$(arg prefix)front_caster_wheel">
+    <material>
+      <ambient>0 0 0 1</ambient>
+      <diffuse>0 0 0 1</diffuse>
+      <specular>0 0 0 1</specular>
+    </material>
+    <mu1>0.0001</mu1>
+    <mu2>0.0001</mu2>
+  </gazebo>
+  <!-- =========================================================
+       REAR CASTER WHEEL
+       ========================================================= -->
+  <joint
+    name="$(arg prefix)back_caster_wheel_joint"
+    type="fixed">
+    <parent link="$(arg prefix)base_link"/>
+    <child link="$(arg prefix)back_caster_wheel"/>
+    <!-- Same position as original articubot_two -->
+    <origin
+      xyz="-0.12 0 0"
+      rpy="0 0 0"/>
+  </joint>
+  <link name="$(arg prefix)back_caster_wheel">
+    <!-- VISUAL -->
+    <visual>
+      <origin
+        xyz="0 0 0"
+        rpy="0 0 0"/>
+      <geometry>
+        <sphere
+          radius="0.01495"/>
+      </geometry>
+      <material name="caster_black">
+        <color
+          rgba="0 0 0 1"/>
+      </material>
+    </visual>
+    <!-- COLLISION -->
+    <collision>
+      <origin
+        xyz="0 0 0"
+        rpy="0 0 0"/>
+      <geometry>
+        <sphere
+          radius="0.01495"/>
+      </geometry>
+    </collision>
+    <!-- INERTIAL -->
+    <inertial>
+      <origin
+        xyz="0 0 0"
+        rpy="0 0 0"/>
+      <mass
+        value="0.1"/>
+      <inertia
+        ixx="${(2.0/5.0) * 0.1 * 0.01495 * 0.01495}"
+        ixy="0"
+        ixz="0"
+        iyy="${(2.0/5.0) * 0.1 * 0.01495 * 0.01495}"
+        iyz="0"
+        izz="${(2.0/5.0) * 0.1 * 0.01495 * 0.01495}"/>
+    </inertial>
+  </link>
+  <!-- GAZEBO -->
+  <gazebo
+    reference="$(arg prefix)back_caster_wheel">
+    <material>
+      <ambient>0 0 0 1</ambient>
+      <diffuse>0 0 0 1</diffuse>
+      <specular>0 0 0 1</specular>
+    </material>
+    <mu1>0.0001</mu1>
+    <mu2>0.0001</mu2>
+  </gazebo>
 </robot>
