Commit message: added robot visual urdf need to add c0ollison and inertial prop

File: benzene_description/urdf/sensors/lidar.urdf.xacro (robot description, xacro)
@@ -1,46 +1,77 @@
 <?xml version="1.0"?>
 <robot xmlns:xacro="http://www.ros.org/wiki/xacro">
-  <xacro:property name="M_PI" value="3.1415926535897931" />
-  <xacro:macro name="lidar_sensor" params="
-    prefix:=''
-    parent:='base_link'
-    frame_id:='laser_frame'
-    mesh_file:='file://$(find benzene_description)/meshes/rplidar/lidar.stl'
-    xyz_offset:='0 0 0.0825'
-    rpy_offset:='0 0 0'
-    mesh_xyz_offset:='0 0 0'
-    mesh_rpy_offset:='${-M_PI/2} 0 0'
-    mesh_scale:='0.001 0.001 0.001'
-    collision_xyz_offset:='0 0 0'
-    collision_rpy_offset:='0 0 0'
-    inertial_xyz_offset:='0 0 0'
-    inertial_rpy_offset:='0 0 0'
-    lidar_width:=0.077
-    lidar_height:=0.0398
-    mass:=0.185
-    material_name:='rplidar_black'
-    material_color:='0.1 0.1 0.1 1'
-    gazebo_material_ambient:='0.1 0.1 0.1 1'
-    gazebo_material_diffuse:='0.1 0.1 0.1 1'
-    gazebo_material_specular:='0.1 0.1 0.1 1'
-    update_rate:=10
-    ray_count:=720
-    min_angle:='-3.14159'
-    max_angle:='3.14159'
-    min_range:='0.20'
-    max_range:='30.0'
-    range_resolution:='0.013'
-    topic_name:='scan'
-    always_on:=true
-    visualize:=false
-    enable_collision:=false">
-    <xacro:property name="radius" value="${lidar_width/2}" />
-    <xacro:property name="ixx_iyy" value="${(mass/12) * (3 * radius * radius + lidar_height * lidar_height)}" />
-    <xacro:property name="izz" value="${(mass/2) * (radius * radius)}" />
+  <!-- =========================================================
+       CONSTANTS
+       ========================================================= -->
+  <xacro:property
+    name="M_PI"
+    value="3.1415926535897931"/>
+  <!-- =========================================================
+       LIDAR MACRO
+       ========================================================= -->
+  <xacro:macro
+    name="lidar_sensor"
+    params="
+      prefix:=''
+      parent:='base_link'
+      frame_id:='laser_frame'
+      mesh_file:='file://$(find benzene_description)/meshes/rplidar/lidar.stl'
+      xyz_offset:='-0.06 0 0.096'
+      rpy_offset:='0 0 0'
+      mesh_xyz_offset:='0 0 0'
+      mesh_rpy_offset:='-1.5707963267948966 0 0'
+      mesh_scale:='0.001 0.001 0.001'
+      collision_xyz_offset:='0 0 0'
+      collision_rpy_offset:='0 0 0'
+      inertial_xyz_offset:='0 0 0'
+      inertial_rpy_offset:='0 0 0'
+      lidar_width:=0.077
+      lidar_height:=0.0398
+      mass:=0.185
+      material_name:='lidar_red'
+      material_color:='1 0 0 1'
+      gazebo_material_ambient:='0.1 0.1 0.1 1'
+      gazebo_material_diffuse:='0.1 0.1 0.1 1'
+      gazebo_material_specular:='0.1 0.1 0.1 1'
+      update_rate:=10
+      ray_count:=360
+      min_angle:='-3.14'
+      max_angle:='3.14'
+      min_range:='0.3'
+      max_range:='12.0'
+      range_resolution:='0.013'
+      topic_name:='scan'
+      always_on:=true
+      visualize:=false
+      enable_collision:=true
+    ">
+    <!-- =======================================================
+         LIDAR INERTIA
+         ======================================================= -->
+    <xacro:property
+      name="radius"
+      value="${lidar_width / 2}"/>
+    <xacro:property
+      name="ixx_iyy"
+      value="${(mass / 12) * (3 * radius * radius + lidar_height * lidar_height)}"/>
+    <xacro:property
+      name="izz"
+      value="${(mass / 2) * (radius * radius)}"/>
+    <!-- =======================================================
+         LIDAR LINK
+         ======================================================= -->
     <link name="${prefix}${frame_id}">
       <visual>
-        <origin xyz="${mesh_xyz_offset}" rpy="${mesh_rpy_offset}"/>
+        <!--
+          This rotates ONLY the STL mesh.
+          -90 degrees around X
+        -->
+        <origin
+          xyz="${mesh_xyz_offset}"
+          rpy="${mesh_rpy_offset}"/>
         <geometry>
-          <mesh filename="${mesh_file}" scale="${mesh_scale}"/>
+          <mesh
+            filename="${mesh_file}"
+            scale="${mesh_scale}"/>
         </geometry>
         <material name="${material_name}">
@@ -48,15 +79,27 @@
         </material>
       </visual>
+      <!-- =====================================================
+           COLLISION
+           ===================================================== -->
       <xacro:if value="${enable_collision}">
         <collision>
-          <origin xyz="${collision_xyz_offset}" rpy="${collision_rpy_offset}"/>
+          <origin
+            xyz="${collision_xyz_offset}"
+            rpy="${collision_rpy_offset}"/>
           <geometry>
-            <cylinder radius="${lidar_width/2}" length="${lidar_height}"/>
+            <mesh
+              filename="${mesh_file}"
+              scale="${mesh_scale}"/>
           </geometry>
         </collision>
       </xacro:if>
+      <!-- =====================================================
+           INERTIAL
+           ===================================================== -->
       <inertial>
-        <mass value="${mass}" />
-        <origin xyz="${inertial_xyz_offset}" rpy="${inertial_rpy_offset}"/>
+        <mass value="${mass}"/>
+        <origin
+          xyz="${inertial_xyz_offset}"
+          rpy="${inertial_rpy_offset}"/>
         <inertia
           ixx="${ixx_iyy}"
@@ -65,12 +108,28 @@
           iyy="${ixx_iyy}"
           iyz="0.0"
-          izz="${izz}" />
+          izz="${izz}"/>
       </inertial>
     </link>
-    <joint name="${prefix}${frame_id}_joint" type="fixed">
+    <!-- =======================================================
+         LIDAR JOINT
+         ======================================================= -->
+    <joint
+      name="${prefix}${frame_id}_joint"
+      type="fixed">
       <parent link="${prefix}${parent}"/>
-      <child link="${prefix}${frame_id}" />
-      <origin xyz="${xyz_offset}" rpy="${rpy_offset}"/>
+      <child link="${prefix}${frame_id}"/>
+      <!--
+        Global LiDAR position:
+        X = -0.06 m
+        Y =  0.00 m
+        Z =  0.096 m
+      -->
+      <origin
+        xyz="${xyz_offset}"
+        rpy="${rpy_offset}"/>
     </joint>
+    <!-- =======================================================
+         GAZEBO / GZ SIM
+         ======================================================= -->
     <gazebo reference="${prefix}${frame_id}">
       <material>
@@ -79,5 +138,10 @@
         <specular>${gazebo_material_specular}</specular>
       </material>
-      <sensor name="${prefix}lidar_sensor" type="gpu_lidar">
+      <!-- =====================================================
+           GPU LIDAR
+           ===================================================== -->
+      <sensor
+        name="${prefix}lidar_sensor"
+        type="gpu_lidar">
         <topic>${topic_name}</topic>
         <update_rate>${update_rate}</update_rate>
@@ -105,5 +169,7 @@
           </range>
         </ray>
-        <gz_frame_id>${prefix}${frame_id}</gz_frame_id>
+        <gz_frame_id>
+          ${prefix}${frame_id}
+        </gz_frame_id>
       </sensor>
     </gazebo>

Commit message: added robot collision and intertial prop

File: benzene_description/urdf/mech/base.urdf.xacro (robot description, xacro)
@@ -1,4 +1,5 @@
 <?xml version="1.0"?>
 <robot xmlns:xacro="http://www.ros.org/wiki/xacro">
+  <xacro:include filename="$(find benzene_description)/urdf/mech/inertial_macros.xacro" />
   <!-- =========================
        BASE DIMENSIONS
@@ -29,6 +30,7 @@
       <collision>
         <geometry>
-          <box
-            size="${base_length} ${base_width} ${base_height}"/>
+          <mesh
+            filename="file://$(find benzene_description)/meshes/benzene/visual/chassis.stl"
+            scale="0.001 0.001 0.001"/>
         </geometry>
         <origin
@@ -36,17 +38,7 @@
           rpy="0 0 0"/>
       </collision>
-      <inertial>
-        <origin
-          xyz="0 0 0"
-          rpy="0 0 0"/>
-        <mass value="${base_mass}"/>
-        <inertia
-          ixx="${(1/12) * base_mass * (base_width*base_width + base_height*base_height)}"
-          ixy="0"
-          ixz="0"
-          iyy="${(1/12) * base_mass * (base_length*base_length + base_height*base_height)}"
-          iyz="0"
-          izz="${(1/12) * base_mass * (base_length*base_length + base_width*base_width)}"/>
-      </inertial>
+      <xacro:inertial_box mass="1.0" x="0.24" y="0.18" z="0.04">
+            <origin xyz="0 0 0" rpy="0 0 0"/>
+        </xacro:inertial_box>
     </link>
     <!-- BASE FOOTPRINT -> BASE LINK -->

File: benzene_description/urdf/mech/wheel.urdf.xacro (robot description, xacro)
@@ -1,4 +1,5 @@
 <?xml version="1.0"?>
 <robot xmlns:xacro="http://www.ros.org/wiki/xacro">
+    <xacro:include filename="$(find benzene_description)/urdf/mech/inertial_macros.xacro" />
     <!-- =========================================================
          WHEEL PARAMETERS
@@ -45,9 +46,9 @@
                 <origin
                     xyz="0 0 0"
-                    rpy="0 0 0"/>
+                    rpy="${-y_reflect * pi/2} 0 0"/>
                 <geometry>
-                    <cylinder
-                        radius="${wheel_radius}"
-                        length="${wheel_width}"/>
+                    <mesh
+                        filename="file://$(find benzene_description)/meshes/benzene/visual/${side}_wheel.stl"
+                        scale="0.001 0.001 0.001"/>
                 </geometry>
             </collision>
@@ -55,17 +56,7 @@
                  INERTIAL
                  ================================================= -->
-            <inertial>
-                <origin
-                    xyz="0 0 0"
-                    rpy="0 0 0"/>
-                <mass value="${wheel_mass}"/>
-                <inertia
-                    ixx="${(wheel_mass / 12.0) * (3.0 * wheel_radius * wheel_radius + wheel_width * wheel_width)}"
-                    ixy="0.0"
-                    ixz="0.0"
-                    iyy="${(wheel_mass / 2.0) * wheel_radius * wheel_radius}"
-                    iyz="0.0"
-                    izz="${(wheel_mass / 12.0) * (3.0 * wheel_radius * wheel_radius + wheel_width * wheel_width)}"/>
-            </inertial>
+            <xacro:inertial_cylinder mass="0.2" radius="0.07" length="0.02">
+                <origin xyz="0 0 0" rpy="0 0 0"/>
+            </xacro:inertial_cylinder>
         </link>
         <!-- =====================================================

File: benzene_description/urdf/robots/benzene.urdf.xacro (robot description, xacro)
@@ -123,18 +123,7 @@
     </collision>
     <!-- INERTIAL -->
-    <inertial>
-      <origin
-        xyz="0 0 0"
-        rpy="0 0 0"/>
-      <mass
-        value="0.1"/>
-      <inertia
-        ixx="${(2.0/5.0) * 0.1 * 0.01495 * 0.01495}"
-        ixy="0"
-        ixz="0"
-        iyy="${(2.0/5.0) * 0.1 * 0.01495 * 0.01495}"
-        iyz="0"
-        izz="${(2.0/5.0) * 0.1 * 0.01495 * 0.01495}"/>
-    </inertial>
+    <xacro:inertial_sphere mass="0.1" radius="0.01495">
+      <origin xyz="0 0 0" rpy="0 0 0"/>
+    </xacro:inertial_sphere>
   </link>
   <!-- GAZEBO -->
@@ -188,18 +177,7 @@
     </collision>
     <!-- INERTIAL -->
-    <inertial>
-      <origin
-        xyz="0 0 0"
-        rpy="0 0 0"/>
-      <mass
-        value="0.1"/>
-      <inertia
-        ixx="${(2.0/5.0) * 0.1 * 0.01495 * 0.01495}"
-        ixy="0"
-        ixz="0"
-        iyy="${(2.0/5.0) * 0.1 * 0.01495 * 0.01495}"
-        iyz="0"
-        izz="${(2.0/5.0) * 0.1 * 0.01495 * 0.01495}"/>
-    </inertial>
+    <xacro:inertial_sphere mass="0.1" radius="0.01495">
+      <origin xyz="0 0 0" rpy="0 0 0"/>
+    </xacro:inertial_sphere>
   </link>
   <!-- GAZEBO -->
