Commit message: Fixed the lidar scan drift

File: benzene_description/urdf/mech/wheel.urdf.xacro (robot description, xacro)
@@ -9,5 +9,5 @@
     <xacro:property name="wheel_width" value="0.020"/>
     <!-- Distance between left and right wheel centers -->
-    <xacro:property name="wheel_separation" value="0.180"/>
+    <xacro:property name="wheel_separation" value="0.185"/>
     <!-- Wheel position relative to base_link -->
     <xacro:property name="wheel_x_offset" value="0.0"/>

File: benzene_description/urdf/mech/wheel.xacro (robot description, xacro)
@@ -12,5 +12,5 @@
     mesh_xyz_offset:='0 0 0'
     mesh_rpy_offset:='0 0 ${pi/2}'
-    wheel_radius:=0.05
+    wheel_radius:=0.035
     wheel_width:=0.03
     wheel_mass:=0.5

File: benzene_hardware/description/urdf/diffbot_description.urdf.xacro (robot description, xacro)
@@ -10,5 +10,5 @@
   <xacro:property name="wheel_mass" value="0.3" /> <!-- arbitrary value for wheel mass -->
   <xacro:property name="wheel_len" value="0.020" />
-  <xacro:property name="wheel_radius" value="0.015" />
+  <xacro:property name="wheel_radius" value="0.035" />
   <xacro:property name="caster_wheel_mass" value="0.1" /> <!-- arbitrary value for caster wheel mass -->
   <xacro:property name="caster_wheel_radius" value="0.015" />
