Commit message: Added benzene new urdf matching to the real robot

File: benzene_description/urdf/control/benzene_control.urdf.xacro (robot description, xacro)
@@ -15,5 +15,5 @@
                     <param name="baud_rate">57600</param>
                     <param name="timeout_ms">1000</param>
-                    <param name="enc_counts_per_rev">1420</param>
+                    <param name="enc_counts_per_rev">1557</param>
                 </xacro:unless>
             </hardware>

File: benzene_description/urdf/robots/benzene.urdf.xacro (robot description, xacro)
@@ -1,147 +1,197 @@
 <?xml version="1.0"?>
-<robot
-  xmlns:xacro="http://www.ros.org/wiki/xacro"
-  name="benzene">
-  <!-- =========================================================
-       CONSTANTS
-       ========================================================= -->
-  <xacro:property
-    name="M_PI"
-    value="3.1415926535897931"/>
-  <!-- =========================================================
-       ARGUMENTS
-       ========================================================= -->
-  <xacro:arg
-    name="robot_name"
-    default="benzene"/>
-  <xacro:arg
-    name="prefix"
-    default=""/>
-  <xacro:arg
-    name="use_gazebo"
-    default="false"/>
-  <!-- =========================================================
-       MECHANICAL COMPONENTS
-       ========================================================= -->
-  <xacro:include
-    filename="$(find benzene_description)/urdf/mech/base.urdf.xacro"/>
-  <xacro:include
-    filename="$(find benzene_description)/urdf/mech/wheel.urdf.xacro"/>
-  <!-- =========================================================
-       SENSORS
-       ========================================================= -->
-  <!-- Camera disabled for now -->
-  <xacro:include
-    filename="$(find benzene_description)/urdf/sensors/camera.urdf.xacro"/>
-  <xacro:include
-    filename="$(find benzene_description)/urdf/sensors/lidar.urdf.xacro"/>
-  <xacro:include
-    filename="$(find benzene_description)/urdf/sensors/imu.urdf.xacro"/>
-  <!-- =========================================================
-       BASE
-       ========================================================= -->
-  <xacro:base
-    prefix="$(arg prefix)"/>
-  <!-- =========================================================
-       LEFT DRIVE WHEEL
-       ========================================================= -->
-  <xacro:wheel
-    prefix="$(arg prefix)"
-    side="left"
-    x_reflect="1"
-    y_reflect="1"/>
-  <!-- =========================================================
-       RIGHT DRIVE WHEEL
-       ========================================================= -->
-  <xacro:wheel
-    prefix="$(arg prefix)"
-    side="right"
-    x_reflect="1"
-    y_reflect="-1"/>
-  <!-- =========================================================
-       LIDAR
-       ========================================================= -->
-  <xacro:lidar_sensor
-    prefix="$(arg prefix)"
-    parent="base_link"
-    frame_id="laser_frame"
-    xyz_offset="-0.06 0 0.096"
-    rpy_offset="0 0 0"
-    mesh_xyz_offset="0 0 0"
-    mesh_rpy_offset="0 0 0"
-    topic_name="scan"/>
-  <!-- =========================================================
-       IMU
-       ========================================================= -->
-  <xacro:imu_sensor
-    prefix="$(arg prefix)"
-    parent="base_link"
-    frame_id="imu"
-    xyz_offset="0 0 0.006"
-    rpy_offset="0 0 0"
-    update_rate="15.0"
-    topic_name="imu/data"/>
-  <!-- =========================================================
-       CAMERA
-       ========================================================= -->
-  <xacro:rgb_camera
-    camera_name="camera"
-    parent="base_link"
-    xyz_offset="0.15 0 0.08"
-    rpy_offset="0 0 0"
-    image_width="640"
-    image_height="480"
-    horizontal_fov="1.089"
-    update_rate="10"
-    clip_near="0.05"
-    clip_far="8.0"
-    topic="cam_1/image_raw"
-    camera_info_topic="cam_1/camera_info"/>
-  <!-- =========================================================
-       FRONT CASTER WHEEL
-       ========================================================= -->
-  <joint
-    name="$(arg prefix)front_caster_wheel_joint"
-    type="fixed">
-    <parent link="$(arg prefix)base_link"/>
-    <child link="$(arg prefix)front_caster_wheel"/>
-    <!-- Same position as original articubot_two -->
-    <origin
-      xyz="0.12 0 0"
-      rpy="0 0 0"/>
-  </joint>
-  <link name="$(arg prefix)front_caster_wheel">
-    <!-- VISUAL -->
+<robot name="benzene" xmlns:xacro="http://www.ros.org/wiki/xacro">
+  <xacro:arg name="robot_name" default="benzene"/>
+  <xacro:arg name="prefix" default=""/>
+  <xacro:arg name="use_gazebo" default="false"/>
+  <xacro:property name="base_length" value="0.340"/>
+  <xacro:property name="base_width"  value="0.240"/>
+  <xacro:property name="base_height" value="0.08"/>
+  <xacro:property name="base_mass"   value="5.0"/>
+  <xacro:property name="wheel_radius" value="0.035"/>
+  <xacro:property name="wheel_width"  value="0.020"/>
+  <xacro:property name="wheel_mass"   value="0.20"/>
+  <xacro:property name="caster_radius" value="0.015"/>
+  <xacro:property name="caster_width"  value="0.020"/>
+  <xacro:property name="caster_mass"   value="0.05"/>
+  <material name="black">
+    <color rgba="0.0 0.0 0.0 1.0"/>
+  </material>
+  <material name="white">
+    <color rgba="1.0 1.0 1.0 1.0"/>
+  </material>
+  <material name="red">
+    <color rgba="1.0 0.0 0.0 1.0"/>
+  </material>
+  <material name="blue">
+    <color rgba="0 0 0.8 1"/>
+  </material>
+  <xacro:macro name="default_inertial" params="mass">
+    <inertial>
+      <mass value="${mass}" />
+      <inertia ixx="1e-3" ixy="0.0" ixz="0.0" iyy="1e-3" iyz="0.0" izz="1e-3" />
+    </inertial>
+  </xacro:macro>
+  <joint name="base_footprint_joint" type="fixed">
+    <parent link="base_footprint"/>
+    <child link="base_link"/>
+    <origin xyz="0 0 0" rpy="0 0 0"/>
+  </joint>
+  <link name="base_footprint"/>
+  <link name="base_link">
     <visual>
-      <origin
-        xyz="0 0 0"
-        rpy="0 0 0"/>
-      <geometry>
-        <sphere
-          radius="0.01495"/>
-      </geometry>
-      <material name="caster_black">
-        <color
-          rgba="0 0 0 1"/>
-      </material>
+      <origin xyz="0 0 0" rpy="1.5708 0 ${pi/2}"/>
+      <geometry>
+        <mesh
+          filename="package://benzene_description/meshes/v3/visual/base_link.stl"
+          scale="0.001 0.001 0.001"/>
+      </geometry>
+      <material name="white"/>
     </visual>
-    <!-- COLLISION -->
     <collision>
-      <origin
-        xyz="0 0 0"
-        rpy="0 0 0"/>
-      <geometry>
-        <sphere
-          radius="0.01495"/>
+      <origin xyz="0 0 0.04" rpy="0 0 0"/>
+      <geometry>
+        <box size="${base_length} ${base_width} ${base_height}"/>
       </geometry>
     </collision>
-    <!-- INERTIAL -->
-    <xacro:inertial_sphere mass="0.1" radius="0.01495">
-      <origin xyz="0 0 0" rpy="0 0 0"/>
-    </xacro:inertial_sphere>
-  </link>
-  <!-- GAZEBO -->
-  <gazebo
-    reference="$(arg prefix)front_caster_wheel">
+    <inertial>
+      <origin xyz="0 0 0" rpy="0 0 0"/>
+      <mass value="${base_mass}"/>
+      <inertia
+        ixx="${(1.0/12.0) * base_mass * (base_width*base_width + base_height*base_height)}"
+        ixy="0.0" ixz="0.0"
+        iyy="${(1.0/12.0) * base_mass * (base_length*base_length + base_height*base_height)}"
+        iyz="0.0"
+        izz="${(1.0/12.0) * base_mass * (base_length*base_length + base_width*base_width)}"/>
+    </inertial>
+  </link>
+  <joint name="right_wheel_joint" type="continuous">
+    <parent link="base_link"/>
+    <child link="right_wheel_link"/>
+    <origin xyz="0 -0.0925 0.020" rpy="0 0 0"/>
+    <axis xyz="0 1 0"/>
+    <dynamics damping="0.05" friction="0.05"/>
+  </joint>
+  <link name="right_wheel_link">
+      <visual>
+        <origin xyz="0 0 0" rpy="0 0 ${pi/2}"/>
+        <geometry>
+          <mesh filename="package://benzene_description/meshes/v3/visual/wheel_link.stl" scale="0.001 0.001 0.001"/>
+        </geometry>
+        <material name="black"/>
+      </visual>
+      <collision>
+        <origin xyz="0 0 0" rpy="-${pi/2} 0 0"/>
+        <geometry>
+          <cylinder
+            radius="${wheel_radius}"
+            length="${wheel_width}"/>
+        </geometry>
+      </collision>
+      <inertial>
+        <origin xyz="0 0 0" rpy="0 0 0"/>
+        <mass value="${wheel_mass}"/>
+        <inertia
+          ixx="${(1.0/12.0) * wheel_mass * (3*wheel_radius*wheel_radius + wheel_width*wheel_width)}"
+          ixy="0.0" ixz="0.0"
+          iyy="${(1.0/12.0) * wheel_mass * (3*wheel_radius*wheel_radius + wheel_width*wheel_width)}"
+          iyz="0.0"
+          izz="${0.5 * wheel_mass * wheel_radius*wheel_radius}"/>
+      </inertial>
+  </link>
+  <joint name="left_wheel_joint" type="continuous">
+    <parent link="base_link"/>
+    <child link="left_wheel_link"/>
+    <origin xyz="0 0.0925 0.020" rpy="0 0 0"/>
+    <axis xyz="0 1 0"/>
+    <dynamics damping="0.05" friction="0.05"/>
+  </joint>
+  <link name="left_wheel_link">
+      <visual>
+        <origin xyz="0 0 0" rpy="0 0 ${pi/2}"/>
+        <geometry>
+          <mesh filename="package://benzene_description/meshes/v3/visual/wheel_link.stl" scale="0.001 0.001 0.001"/>
+        </geometry>
+        <material name="black"/>
+      </visual>
+      <collision>
+        <origin xyz="0 0 0" rpy="-${pi/2} 0 0"/>
+        <geometry>
+          <cylinder
+            radius="${wheel_radius}"
+            length="${wheel_width}"/>
+        </geometry>
+      </collision>
+      <inertial>
+        <origin xyz="0 0 0" rpy="0 0 0"/>
+        <mass value="${wheel_mass}"/>
+        <inertia
+          ixx="${(1.0/12.0) * wheel_mass * (3*wheel_radius*wheel_radius + wheel_width*wheel_width)}"
+          ixy="0.0" ixz="0.0"
+          iyy="${(1.0/12.0) * wheel_mass * (3*wheel_radius*wheel_radius + wheel_width*wheel_width)}"
+          iyz="0.0"
+          izz="${0.5 * wheel_mass * wheel_radius*wheel_radius}"/>
+      </inertial>
+  </link>
+  <joint name="back_caster_wheel_joint" type="fixed">
+    <parent link="base_link"/>
+    <child link="back_caster_wheel"/>
+    <origin xyz="-0.13 0 0" rpy="0 0 0"/>
+  </joint>
+  <link name="back_caster_wheel">
+    <visual>
+      <origin xyz="0 0 0" rpy="0 0 0"/>
+      <geometry>
+        <mesh filename="package://benzene_description/meshes/v3/visual/caster_link.stl" scale="0.001 0.001 0.001"/>
+      </geometry>
+      <material name="black"/>
+    </visual>
+    <collision>
+      <origin xyz="0 0 0" rpy="0 0 0"/>
+      <geometry>
+        <sphere radius="${caster_radius}"/>
+      </geometry>
+    </collision>
+    <inertial>
+      <origin xyz="0 0 0" rpy="0 0 0"/>
+      <mass value="${caster_mass}"/>
+      <inertia
+        ixx="${(2.0/5.0) * caster_mass * caster_radius * caster_radius}"
+        ixy="0.0" ixz="0.0"
+        iyy="${(2.0/5.0) * caster_mass * caster_radius * caster_radius}"
+        iyz="0.0"
+        izz="${(2.0/5.0) * caster_mass * caster_radius * caster_radius}"/>
+    </inertial>
+  </link>
+  <joint name="front_caster_wheel_joint" type="fixed">
+    <parent link="base_link"/>
+    <child link="front_caster_wheel"/>
+    <origin xyz="0.13 0 0" rpy="0 0 0"/>
+  </joint>
+  <link name="front_caster_wheel">
+    <visual>
+      <origin xyz="0 0 0" rpy="0 0 0"/>
+      <geometry>
+        <mesh filename="package://benzene_description/meshes/v3/visual/caster_link.stl" scale="0.001 0.001 0.001"/>
+      </geometry>
+      <material name="black"/>
+    </visual>
+    <collision>
+      <origin xyz="0 0 0" rpy="0 0 0"/>
+      <geometry>
+        <sphere radius="${caster_radius}"/>
+      </geometry>
+    </collision>
+    <inertial>
+      <origin xyz="0 0 0" rpy="0 0 0"/>
+      <mass value="${caster_mass}"/>
+      <inertia
+        ixx="${(2.0/5.0) * caster_mass * caster_radius * caster_radius}"
+        ixy="0.0" ixz="0.0"
+        iyy="${(2.0/5.0) * caster_mass * caster_radius * caster_radius}"
+        iyz="0.0"
+        izz="${(2.0/5.0) * caster_mass * caster_radius * caster_radius}"/>
+    </inertial>
+  </link>
+  <gazebo reference="$(arg prefix)front_caster_wheel">
     <material>
       <ambient>0 0 0 1</ambient>
@@ -152,50 +202,54 @@
     <mu2>0.0001</mu2>
   </gazebo>
-  <!-- =========================================================
-       REAR CASTER WHEEL
-       ========================================================= -->
-  <joint
-    name="$(arg prefix)back_caster_wheel_joint"
-    type="fixed">
-    <parent link="$(arg prefix)base_link"/>
-    <child link="$(arg prefix)back_caster_wheel"/>
-    <!-- Same position as original articubot_two -->
-    <origin
-      xyz="-0.12 0 0"
-      rpy="0 0 0"/>
-  </joint>
-  <link name="$(arg prefix)back_caster_wheel">
-    <!-- VISUAL -->
-    <visual>
-      <origin
-        xyz="0 0 0"
-        rpy="0 0 0"/>
-      <geometry>
-        <sphere
-          radius="0.01495"/>
-      </geometry>
-      <material name="caster_black">
-        <color
-          rgba="0 0 0 1"/>
-      </material>
-    </visual>
-    <!-- COLLISION -->
-    <collision>
-      <origin
-        xyz="0 0 0"
-        rpy="0 0 0"/>
-      <geometry>
-        <sphere
-          radius="0.01495"/>
-      </geometry>
-    </collision>
-    <!-- INERTIAL -->
-    <xacro:inertial_sphere mass="0.1" radius="0.01495">
-      <origin xyz="0 0 0" rpy="0 0 0"/>
-    </xacro:inertial_sphere>
-  </link>
-  <!-- GAZEBO -->
-  <gazebo
-    reference="$(arg prefix)back_caster_wheel">
+  <!-- ===========================================================
+       SENSOR MACROS (lidar / camera / imu) — each brings its own
+       link, fixed joint, and <gazebo><sensor> plugin block.
+       Adjust these include paths to wherever the files actually
+       live in benzene_description (e.g. urdf/sensors/...).
+       =========================================================== -->
+  <xacro:include filename="$(find benzene_description)/urdf/sensors/lidar.urdf.xacro"/>
+  <xacro:include filename="$(find benzene_description)/urdf/sensors/simple_camera.urdf.xacro"/>
+  <xacro:include filename="$(find benzene_description)/urdf/sensors/imu.urdf.xacro"/>
+  <xacro:lidar_sensor
+    prefix="$(arg prefix)"
+    parent="base_link"
+    frame_id="laser_frame"
+    xyz_offset="0 0 0.08"
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
File: benzene_description/urdf/sensors/imu.urdf.xacro (robot description, xacro)
@@ -11,7 +11,7 @@
         inertial_rpy_offset:='0 0 0'
         mass:=0.031
-        length:=0.03899
-        width:=0.03785
-        height:=0.01338
+        length:=0.0164
+        width:=0.0212
+        height:=0.0033
         material_name:='imu_black'
         material_color:='0.1 0.1 0.1 1'

File: benzene_description/urdf/sensors/lidar.urdf.xacro (robot description, xacro)
@@ -17,8 +17,8 @@
       frame_id:='laser_frame'
       mesh_file:='file://$(find benzene_description)/meshes/rplidar/lidar.stl'
-      xyz_offset:='-0.06 0 0.096'
+      xyz_offset:='0 0 0'
       rpy_offset:='0 0 0'
       mesh_xyz_offset:='0 0 0'
-      mesh_rpy_offset:='-1.5707963267948966 0 0'
+      mesh_rpy_offset:='0 0 0'
       mesh_scale:='0.001 0.001 0.001'
       collision_xyz_offset:='0 0 0'

File: benzene_description/urdf/sensors/simple_camera.urdf.xacro (robot description, xacro)
@@ -2,18 +2,15 @@
 <robot xmlns:xacro="http://www.ros.org/wiki/xacro">
   <xacro:property name="M_PI" value="3.1415926535897931"/>
-  <xacro:macro name="rgb_camera" params="
+  <xacro:macro name="simple_camera" params="
     prefix:=''
     camera_name:='camera'
     parent:='base_link'
-    xyz_offset:='0.015 0 0.08'
+    xyz_offset:='0 0 0'
     rpy_offset:='0 0 0'
-    mesh_file:=''
-    mesh_xyz_offset:='0 0 0'
-    mesh_rpy_offset:='0 0 0'
-    cam_width:=0.03
-    cam_height:=0.03
+    cam_width:=0.025
+    cam_height:=0.024
     cam_depth:=0.009
-    material_name:='red'
-    material_color:='1 0 0 1'
+    material_name:='black'
+    material_color:='0.05 0.05 0.05 1'
     horizontal_fov:=1.089
     image_width:=640
@@ -21,29 +18,20 @@
     clip_near:=0.05
     clip_far:=8.0
-    update_rate:=10
+    update_rate:=30
     always_on:=true
     visualize:=true
-    topic:='cam_1/image_raw'
-    camera_info_topic:='cam_1/camera_info'
+    topic:='camera/image_raw'
+    camera_info_topic:='camera/camera_info'
   ">
-    <!-- ========================= -->
     <!-- Camera Body -->
-    <!-- ========================= -->
     <link name="${prefix}${camera_name}_link">
       <visual>
         <origin
-          xyz="${mesh_xyz_offset}"
-          rpy="${mesh_rpy_offset}"/>
-        <xacro:if value="${mesh_file != ''}">
-          <geometry>
-            <mesh filename="${mesh_file}"/>
-          </geometry>
-        </xacro:if>
-        <xacro:unless value="${mesh_file != ''}">
-          <geometry>
-            <box
-              size="${cam_depth} ${cam_width} ${cam_height}"/>
-          </geometry>
-        </xacro:unless>
+          xyz="0 0 0"
+          rpy="0 0 0"/>
+        <geometry>
+          <box
+            size="${cam_depth} ${cam_width} ${cam_height}"/>
+        </geometry>
         <material name="${material_name}">
           <color rgba="${material_color}"/>
@@ -51,7 +39,5 @@
       </visual>
     </link>
-    <!-- ========================= -->
     <!-- Camera Mount Joint -->
-    <!-- ========================= -->
     <joint
       name="${prefix}${camera_name}_joint"
@@ -63,7 +49,6 @@
         rpy="${rpy_offset}"/>
     </joint>
-    <!-- ========================= -->
     <!-- Optical Frame -->
-    <!-- ========================= -->
+    <link name="${prefix}${camera_name}_optical"/>
     <joint
       name="${prefix}${camera_name}_optical_joint"
@@ -75,10 +60,7 @@
         rpy="${-M_PI/2} 0 ${-M_PI/2}"/>
     </joint>
-    <link name="${prefix}${camera_name}_optical"/>
-    <!-- ========================= -->
-    <!-- Gazebo RGB Camera -->
-    <!-- ========================= -->
+    <!-- Gazebo Simple RGB Camera -->
     <gazebo reference="${prefix}${camera_name}_link">
-      <material>Gazebo/Red</material>
+      <material>Gazebo/Black</material>
       <sensor
         name="${prefix}${camera_name}"
@@ -89,5 +71,4 @@
         <update_rate>${update_rate}</update_rate>
         <camera>
-          <camera_info_topic>${camera_info_topic}</camera_info_topic>
           <horizontal_fov>${horizontal_fov}</horizontal_fov>
           <image>

Commit message: Updated cnts also some work in hardware interface

File: benzene_description/urdf/control/benzene_control.urdf.xacro (robot description, xacro)
@@ -15,5 +15,5 @@
                     <param name="baud_rate">57600</param>
                     <param name="timeout_ms">1000</param>
-                    <param name="enc_counts_per_rev">1557</param>
+                    <param name="enc_counts_per_rev">1559</param>
                 </xacro:unless>
             </hardware>

File: benzene_hardware/description/ros2_control/diffbot.ros2_control.xacro (robot description, xacro)
@@ -1,19 +1,25 @@
 <?xml version="1.0"?>
 <robot xmlns:xacro="http://www.ros.org/wiki/xacro">
-  <xacro:macro name="diffbot_ros2_control" params="name prefix">
+  <xacro:macro name="diffbot_ros2_control" params="name prefix use_mock:=false">
     <ros2_control name="${name}" type="system">
       <hardware>
-        <plugin>diffdrive_arduino/DiffDriveArduinoHardware</plugin>
-        <param name="left_wheel_name">left_wheel_joint</param>
-        <param name="right_wheel_name">right_wheel_joint</param>
-        <param name="loop_rate">30</param>
-        <param name="device">/dev/serial/by-path/platform-fd500000.pcie-pci-0000:01:00.0-usb-0:1.3:1.0-port0</param>
-        <param name="baud_rate">57600</param>
-        <param name="timeout_ms">1000</param>
-        <param name="enc_counts_per_rev">3436</param>
-        <param name="pid_p">20</param>
-        <param name="pid_d">12</param>
-        <param name="pid_i">0</param>
-        <param name="pid_o">50</param>
+        <xacro:if value="${use_mock}">
+          <plugin>mock_components/GenericSystem</plugin>
+          <param name="calculate_dynamics">true</param>
+        </xacro:if>
+        <xacro:unless value="${use_mock}">
+          <plugin>diffdrive_arduino/DiffDriveArduinoHardware</plugin>
+          <param name="left_wheel_name">left_wheel_joint</param>
+          <param name="right_wheel_name">right_wheel_joint</param>
+          <param name="loop_rate">30</param>
+          <param name="device">/dev/serial/by-path/platform-fd500000.pcie-pci-0000:01:00.0-usb-0:1.3:1.0-port0</param>
+          <param name="baud_rate">57600</param>
+          <param name="timeout_ms">1000</param>
+          <param name="enc_counts_per_rev">1559</param>
+          <param name="pid_p">2</param>
+          <param name="pid_d">0</param>
+          <param name="pid_i">0</param>
+          <param name="pid_o">50</param>
+        </xacro:unless>
       </hardware>
       <joint name="${prefix}left_wheel_joint">

File: benzene_hardware/description/urdf/diffbot.urdf.xacro (robot description, xacro)
@@ -3,11 +3,12 @@
 <robot xmlns:xacro="http://www.ros.org/wiki/xacro" name="diffdrive_robot">
   <xacro:arg name="prefix" default="" />
-  <xacro:include filename="$(find diffdrive_arduino)/urdf/diffbot_description.urdf.xacro" />
+  <xacro:arg name="use_mock" default="false" />
+  <xacro:include filename="$(find benzene_hardware)/urdf/diffbot_description.urdf.xacro" />
   <!-- Import Rviz colors -->
-  <xacro:include filename="$(find diffdrive_arduino)/urdf/diffbot.materials.xacro" />
+  <xacro:include filename="$(find benzene_hardware)/urdf/diffbot.materials.xacro" />
   <!-- Import diffbot ros2_control description -->
-  <xacro:include filename="$(find diffdrive_arduino)/ros2_control/diffbot.ros2_control.xacro" />
+  <xacro:include filename="$(find benzene_hardware)/ros2_control/diffbot.ros2_control.xacro" />
   <xacro:diffbot prefix="$(arg prefix)" />
   <xacro:diffbot_ros2_control
-    name="DiffBot" prefix="$(arg prefix)" />
+    name="DiffBot" prefix="$(arg prefix)" use_mock="$(arg use_mock)" />
 </robot>
