Commit message: Added test scripts to navigation, also added camera to work with

File: benzene_description/urdf/robots/benzene.urdf.xacro (robot description, xacro)
@@ -32,8 +32,6 @@
        ========================================================= -->
   <!-- Camera disabled for now -->
-  <!--
   <xacro:include
     filename="$(find benzene_description)/urdf/sensors/camera.urdf.xacro"/>
-  -->
   <xacro:include
     filename="$(find benzene_description)/urdf/sensors/lidar.urdf.xacro"/>
@@ -84,4 +82,20 @@
     update_rate="15.0"
     topic_name="imu/data"/>
+  <!-- =========================================================
+       CAMERA
+       ========================================================= -->
+  <xacro:rgb_camera
+    camera_name="camera"
+    parent="base_link"
+    xyz_offset="0.15 0 0.08"
+    rpy_offset="0 0 0"
+    image_width="640"
+    image_height="480"
+    horizontal_fov="1.089"
+    update_rate="10"
+    clip_near="0.05"
+    clip_far="8.0"
+    topic="cam_1/image_raw"
+    camera_info_topic="cam_1/camera_info"/>
   <!-- =========================================================
        FRONT CASTER WHEEL

File: benzene_description/urdf/sensors/camera.urdf.xacro (robot description, xacro)
@@ -1,132 +1,96 @@
 <?xml version="1.0"?>
 <robot xmlns:xacro="http://www.ros.org/wiki/xacro">
-  <xacro:property name="M_PI" value="3.1415926535897931" />
-  <xacro:macro name="rgbd_camera" params="
+  <xacro:property name="M_PI" value="3.1415926535897931"/>
+  <xacro:macro name="rgb_camera" params="
     prefix:=''
-    camera_name:='cam_1'
+    camera_name:='camera'
     parent:='base_link'
-    mesh_file:='file://$(find yahboom_rosmaster_description)/meshes/intel_realsense/visual/d435.stl'
-    xyz_offset:='0.105 0 0.05'
-    rpy_offset:='0 -0.50 0'
+    xyz_offset:='0.15 0 0.08'
+    rpy_offset:='0 0 0'
+    mesh_file:=''
     mesh_xyz_offset:='0 0 0'
-    mesh_rpy_offset:='${M_PI/2} 0.0 ${M_PI/2}'
-    collision_xyz_offset:='0 0 0'
-    collision_rpy_offset:='0 0 0'
-    inertial_xyz_offset:='0 0 0'
-    inertial_rpy_offset:='0 0 0'
-    optical_xyz_offset:='0 0 0'
-    optical_rpy_offset:='${-M_PI/2} 0 ${-M_PI/2}'
-    depth_frame_xyz_offset:='0 0 0'
-    depth_frame_rpy_offset:='0 0 0'
-    infra1_xyz_offset:='0 0 0'
-    infra1_rpy_offset:='0 0 0'
-    infra2_xyz_offset:='0 -0.05 0'
-    infra2_rpy_offset:='0 0 0'
-    color_xyz_offset:='0 0.015 0'
-    color_rpy_offset:='0 0 0'
-    cam_width:=0.090
-    cam_height:=0.025
-    cam_depth:=0.02505
-    mass:=0.072
-    ixx:=0.003881243
-    ixy:=0.0
-    ixz:=0.0
-    iyy:=0.000498940
-    iyz:=0.0
-    izz:=0.003879257
-    material_name:='aluminum'
-    material_color:='0.5 0.5 0.5 1'
-    horizontal_fov:=1.5184
-    image_width:=424
-    image_height:=240
+    mesh_rpy_offset:='0 0 0'
+    cam_width:=0.03
+    cam_height:=0.03
+    cam_depth:=0.009
+    material_name:='red'
+    material_color:='1 0 0 1'
+    horizontal_fov:=1.089
+    image_width:=640
+    image_height:=480
     clip_near:=0.05
-    clip_far:=1.5
-    update_rate:=2
-    always_on:=1
+    clip_far:=8.0
+    update_rate:=10
+    always_on:=true
     visualize:=true
-    enable_collision:=false">
+    topic:='cam_1/image_raw'
+    camera_info_topic:='cam_1/camera_info'
+  ">
+    <!-- ========================= -->
+    <!-- Camera Body -->
+    <!-- ========================= -->
     <link name="${prefix}${camera_name}_link">
       <visual>
-        <origin xyz="${mesh_xyz_offset}" rpy="${mesh_rpy_offset}"/>
-        <geometry>
-          <mesh filename="${mesh_file}" />
-        </geometry>
+        <origin
+          xyz="${mesh_xyz_offset}"
+          rpy="${mesh_rpy_offset}"/>
+        <xacro:if value="${mesh_file != ''}">
+          <geometry>
+            <mesh filename="${mesh_file}"/>
+          </geometry>
+        </xacro:if>
+        <xacro:unless value="${mesh_file != ''}">
+          <geometry>
+            <box
+              size="${cam_depth} ${cam_width} ${cam_height}"/>
+          </geometry>
+        </xacro:unless>
         <material name="${material_name}">
           <color rgba="${material_color}"/>
         </material>
       </visual>
-      <xacro:if value="${enable_collision}">
-        <collision>
-          <origin xyz="${collision_xyz_offset}" rpy="${collision_rpy_offset}"/>
-          <geometry>
-            <box size="${cam_depth} ${cam_width} ${cam_height}"/>
-          </geometry>
-        </collision>
-      </xacro:if>
-      <inertial>
-        <mass value="${mass}" />
-        <origin xyz="${inertial_xyz_offset}" rpy="${inertial_rpy_offset}"/>
-        <inertia ixx="${ixx}" ixy="${ixy}" ixz="${ixz}"
-                 iyy="${iyy}" iyz="${iyz}" izz="${izz}" />
-      </inertial>
     </link>
-    <joint name="${prefix}${camera_name}_joint" type="fixed">
+    <!-- ========================= -->
+    <!-- Camera Mount Joint -->
+    <!-- ========================= -->
+    <joint
+      name="${prefix}${camera_name}_joint"
+      type="fixed">
       <parent link="${prefix}${parent}"/>
-      <child link="${prefix}${camera_name}_link" />
-      <origin xyz="${xyz_offset}" rpy="${rpy_offset}"/>
+      <child link="${prefix}${camera_name}_link"/>
+      <origin
+        xyz="${xyz_offset}"
+        rpy="${rpy_offset}"/>
     </joint>
-    <joint name="${prefix}${camera_name}_depth_joint" type="fixed">
-      <origin xyz="${depth_frame_xyz_offset}" rpy="${depth_frame_rpy_offset}"/>
+    <!-- ========================= -->
+    <!-- Optical Frame -->
+    <!-- ========================= -->
+    <joint
+      name="${prefix}${camera_name}_optical_joint"
+      type="fixed">
       <parent link="${prefix}${camera_name}_link"/>
-      <child link="${prefix}${camera_name}_depth_frame" />
+      <child link="${prefix}${camera_name}_optical"/>
+      <origin
+        xyz="0 0 0"
+        rpy="${-M_PI/2} 0 ${-M_PI/2}"/>
     </joint>
-    <link name="${prefix}${camera_name}_depth_frame"/>
-    <joint name="${prefix}${camera_name}_depth_optical_joint" type="fixed">
-      <origin xyz="${optical_xyz_offset}" rpy="${optical_rpy_offset}" />
-      <parent link="${prefix}${camera_name}_depth_frame" />
-      <child link="${prefix}${camera_name}_depth_optical_frame" />
-    </joint>
-    <link name="${prefix}${camera_name}_depth_optical_frame"/>
-    <joint name="${prefix}${camera_name}_infra1_joint" type="fixed">
-      <origin xyz="${infra1_xyz_offset}" rpy="${infra1_rpy_offset}" />
-      <parent link="${prefix}${camera_name}_link" />
-      <child link="${prefix}${camera_name}_infra1_frame" />
-    </joint>
-    <link name="${prefix}${camera_name}_infra1_frame"/>
-    <joint name="${prefix}${camera_name}_infra1_optical_joint" type="fixed">
-      <origin xyz="${optical_xyz_offset}" rpy="${optical_rpy_offset}" />
-      <parent link="${prefix}${camera_name}_infra1_frame" />
-      <child link="${prefix}${camera_name}_infra1_optical_frame" />
-    </joint>
-    <link name="${prefix}${camera_name}_infra1_optical_frame"/>
-    <joint name="${prefix}${camera_name}_infra2_joint" type="fixed">
-      <origin xyz="${infra2_xyz_offset}" rpy="${infra2_rpy_offset}" />
-      <parent link="${prefix}${camera_name}_link" />
-      <child link="${prefix}${camera_name}_infra2_frame" />
-    </joint>
-    <link name="${prefix}${camera_name}_infra2_frame"/>
-    <joint name="${prefix}${camera_name}_infra2_optical_joint" type="fixed">
-      <origin xyz="${optical_xyz_offset}" rpy="${optical_rpy_offset}" />
-      <parent link="${prefix}${camera_name}_infra2_frame" />
-      <child link="${prefix}${camera_name}_infra2_optical_frame" />
-    </joint>
-    <link name="${prefix}${camera_name}_infra2_optical_frame"/>
-    <joint name="${prefix}${camera_name}_color_joint" type="fixed">
-      <origin xyz="${color_xyz_offset}" rpy="${color_rpy_offset}" />
-      <parent link="${prefix}${camera_name}_link" />
-      <child link="${prefix}${camera_name}_color_frame" />
-    </joint>
-    <link name="${prefix}${camera_name}_color_frame"/>
-    <joint name="${prefix}${camera_name}_color_optical_joint" type="fixed">
-      <origin xyz="${optical_xyz_offset}" rpy="${optical_rpy_offset}" />
-      <parent link="${prefix}${camera_name}_color_frame" />
-      <child link="${prefix}${camera_name}_color_optical_frame" />
-    </joint>
-    <link name="${prefix}${camera_name}_color_optical_frame"/>
+    <link name="${prefix}${camera_name}_optical"/>
+    <!-- ========================= -->
+    <!-- Gazebo RGB Camera -->
+    <!-- ========================= -->
     <gazebo reference="${prefix}${camera_name}_link">
-      <sensor name="${prefix}${camera_name}" type="rgbd_camera">
+      <material>Gazebo/Red</material>
+      <sensor
+        name="${prefix}${camera_name}"
+        type="camera">
+        <pose>0 0 0 0 0 0</pose>
+        <always_on>${always_on}</always_on>
+        <visualize>${visualize}</visualize>
+        <update_rate>${update_rate}</update_rate>
         <camera>
+          <camera_info_topic>${camera_info_topic}</camera_info_topic>
           <horizontal_fov>${horizontal_fov}</horizontal_fov>
           <image>
+            <format>R8G8B8</format>
             <width>${image_width}</width>
             <height>${image_height}</height>
@@ -137,9 +101,8 @@
           </clip>
         </camera>
-        <always_on>${always_on}</always_on>
-        <gz_frame_id>${prefix}${camera_name}_depth_optical_frame</gz_frame_id>
-        <topic>${camera_name}</topic>
-        <update_rate>${update_rate}</update_rate>
-        <visualize>${visualize}</visualize>
+        <topic>${topic}</topic>
+        <gz_frame_id>
+          ${prefix}${camera_name}_optical
+        </gz_frame_id>
       </sensor>
     </gazebo>

Commit message: Made URDF clean

File: benzene_description/urdf/robots/benzene.urdf.xacro (robot description, xacro)
@@ -12,203 +12,22 @@
   <xacro:property name="wheel_mass"   value="0.20"/>
   <xacro:property name="caster_radius" value="0.015"/>
-  <xacro:property name="caster_width"  value="0.020"/>
   <xacro:property name="caster_mass"   value="0.05"/>
-  <material name="black">
-    <color rgba="0.0 0.0 0.0 1.0"/>
-  </material>
-  <material name="white">
-    <color rgba="1.0 1.0 1.0 1.0"/>
-  </material>
-  <material name="red">
-    <color rgba="1.0 0.0 0.0 1.0"/>
-  </material>
-  <material name="blue">
-    <color rgba="0 0 0.8 1"/>
-  </material>
-  <xacro:macro name="default_inertial" params="mass">
-    <inertial>
-      <mass value="${mass}" />
-      <inertia ixx="1e-3" ixy="0.0" ixz="0.0" iyy="1e-3" iyz="0.0" izz="1e-3" />
-    </inertial>
-  </xacro:macro>
-  <joint name="base_footprint_joint" type="fixed">
-    <parent link="base_footprint"/>
-    <child link="base_link"/>
-    <origin xyz="0 0 0" rpy="0 0 0"/>
-  </joint>
-  <link name="base_footprint"/>
-  <link name="base_link">
-    <visual>
-      <origin xyz="0 0 0" rpy="1.5708 0 ${pi/2}"/>
-      <geometry>
-        <mesh
-          filename="package://benzene_description/meshes/v3/visual/base_link.stl"
-          scale="0.001 0.001 0.001"/>
-      </geometry>
-      <material name="white"/>
-    </visual>
-    <collision>
-      <origin xyz="0 0 0.04" rpy="0 0 0"/>
-      <geometry>
-        <box size="${base_length} ${base_width} ${base_height}"/>
-      </geometry>
-    </collision>
-    <inertial>
-      <origin xyz="0 0 0" rpy="0 0 0"/>
-      <mass value="${base_mass}"/>
-      <inertia
-        ixx="${(1.0/12.0) * base_mass * (base_width*base_width + base_height*base_height)}"
-        ixy="0.0" ixz="0.0"
-        iyy="${(1.0/12.0) * base_mass * (base_length*base_length + base_height*base_height)}"
-        iyz="0.0"
-        izz="${(1.0/12.0) * base_mass * (base_length*base_length + base_width*base_width)}"/>
-    </inertial>
-  </link>
-  <joint name="right_wheel_joint" type="continuous">
-    <parent link="base_link"/>
-    <child link="right_wheel_link"/>
-    <origin xyz="0 -0.0925 0.020" rpy="0 0 0"/>
-    <axis xyz="0 1 0"/>
-    <dynamics damping="0.05" friction="0.05"/>
-  </joint>
-  <link name="right_wheel_link">
-      <visual>
-        <origin xyz="0 0 0" rpy="0 0 ${pi/2}"/>
-        <geometry>
-          <mesh filename="package://benzene_description/meshes/v3/visual/wheel_link.stl" scale="0.001 0.001 0.001"/>
-        </geometry>
-        <material name="black"/>
-      </visual>
-      <collision>
-        <origin xyz="0 0 0" rpy="-${pi/2} 0 0"/>
-        <geometry>
-          <cylinder
-            radius="${wheel_radius}"
-            length="${wheel_width}"/>
-        </geometry>
-      </collision>
-      <inertial>
-        <origin xyz="0 0 0" rpy="0 0 0"/>
-        <mass value="${wheel_mass}"/>
-        <inertia
-          ixx="${(1.0/12.0) * wheel_mass * (3*wheel_radius*wheel_radius + wheel_width*wheel_width)}"
-          ixy="0.0" ixz="0.0"
-          iyy="${(1.0/12.0) * wheel_mass * (3*wheel_radius*wheel_radius + wheel_width*wheel_width)}"
-          iyz="0.0"
-          izz="${0.5 * wheel_mass * wheel_radius*wheel_radius}"/>
-      </inertial>
-  </link>
-  <joint name="left_wheel_joint" type="continuous">
-    <parent link="base_link"/>
-    <child link="left_wheel_link"/>
-    <origin xyz="0 0.0925 0.020" rpy="0 0 0"/>
-    <axis xyz="0 1 0"/>
-    <dynamics damping="0.05" friction="0.05"/>
-  </joint>
-  <link name="left_wheel_link">
-      <visual>
-        <origin xyz="0 0 0" rpy="0 0 ${pi/2}"/>
-        <geometry>
-          <mesh filename="package://benzene_description/meshes/v3/visual/wheel_link.stl" scale="0.001 0.001 0.001"/>
-        </geometry>
-        <material name="black"/>
-      </visual>
-      <collision>
-        <origin xyz="0 0 0" rpy="-${pi/2} 0 0"/>
-        <geometry>
-          <cylinder
-            radius="${wheel_radius}"
-            length="${wheel_width}"/>
-        </geometry>
-      </collision>
-      <inertial>
-        <origin xyz="0 0 0" rpy="0 0 0"/>
-        <mass value="${wheel_mass}"/>
-        <inertia
-          ixx="${(1.0/12.0) * wheel_mass * (3*wheel_radius*wheel_radius + wheel_width*wheel_width)}"
-          ixy="0.0" ixz="0.0"
-          iyy="${(1.0/12.0) * wheel_mass * (3*wheel_radius*wheel_radius + wheel_width*wheel_width)}"
-          iyz="0.0"
-          izz="${0.5 * wheel_mass * wheel_radius*wheel_radius}"/>
-      </inertial>
-  </link>
-  <joint name="back_caster_wheel_joint" type="fixed">
-    <parent link="base_link"/>
-    <child link="back_caster_wheel"/>
-    <origin xyz="-0.13 0 0" rpy="0 0 0"/>
-  </joint>
-  <link name="back_caster_wheel">
-    <visual>
-      <origin xyz="0 0 0" rpy="0 0 0"/>
-      <geometry>
-        <mesh filename="package://benzene_description/meshes/v3/visual/caster_link.stl" scale="0.001 0.001 0.001"/>
-      </geometry>
-      <material name="black"/>
-    </visual>
-    <collision>
-      <origin xyz="0 0 0" rpy="0 0 0"/>
-      <geometry>
-        <sphere radius="${caster_radius}"/>
-      </geometry>
-    </collision>
-    <inertial>
-      <origin xyz="0 0 0" rpy="0 0 0"/>
-      <mass value="${caster_mass}"/>
-      <inertia
-        ixx="${(2.0/5.0) * caster_mass * caster_radius * caster_radius}"
-        ixy="0.0" ixz="0.0"
-        iyy="${(2.0/5.0) * caster_mass * caster_radius * caster_radius}"
-        iyz="0.0"
-        izz="${(2.0/5.0) * caster_mass * caster_radius * caster_radius}"/>
-    </inertial>
-  </link>
-  <joint name="front_caster_wheel_joint" type="fixed">
-    <parent link="base_link"/>
-    <child link="front_caster_wheel"/>
-    <origin xyz="0.13 0 0" rpy="0 0 0"/>
-  </joint>
-  <link name="front_caster_wheel">
-    <visual>
-      <origin xyz="0 0 0" rpy="0 0 0"/>
-      <geometry>
-        <mesh filename="package://benzene_description/meshes/v3/visual/caster_link.stl" scale="0.001 0.001 0.001"/>
-      </geometry>
-      <material name="black"/>
-    </visual>
-    <collision>
-      <origin xyz="0 0 0" rpy="0 0 0"/>
-      <geometry>
-        <sphere radius="${caster_radius}"/>
-      </geometry>
-    </collision>
-    <inertial>
-      <origin xyz="0 0 0" rpy="0 0 0"/>
-      <mass value="${caster_mass}"/>
-      <inertia
-        ixx="${(2.0/5.0) * caster_mass * caster_radius * caster_radius}"
-        ixy="0.0" ixz="0.0"
-        iyy="${(2.0/5.0) * caster_mass * caster_radius * caster_radius}"
-        iyz="0.0"
-        izz="${(2.0/5.0) * caster_mass * caster_radius * caster_radius}"/>
-    </inertial>
-  </link>
-  <gazebo reference="$(arg prefix)front_caster_wheel">
-    <material>
-      <ambient>0 0 0 1</ambient>
-      <diffuse>0 0 0 1</diffuse>
-      <specular>0 0 0 1</specular>
-    </material>
-    <mu1>0.0001</mu1>
-    <mu2>0.0001</mu2>
-  </gazebo>
-  <!-- ===========================================================
-       SENSOR MACROS (lidar / camera / imu) — each brings its own
-       link, fixed joint, and <gazebo><sensor> plugin block.
-       Adjust these include paths to wherever the files actually
-       live in benzene_description (e.g. urdf/sensors/...).
-       =========================================================== -->
-  <xacro:include filename="$(find benzene_description)/urdf/sensors/lidar.urdf.xacro"/>
-  <xacro:include filename="$(find benzene_description)/urdf/sensors/simple_camera.urdf.xacro"/>
-  <xacro:include filename="$(find benzene_description)/urdf/sensors/imu.urdf.xacro"/>
+  <xacro:include filename="$(find benzene_description)/urdf/sensors/lidar.xacro"/>
+  <xacro:include filename="$(find benzene_description)/urdf/sensors/simple_camera.xacro"/>
+  <xacro:include filename="$(find benzene_description)/urdf/sensors/imu.xacro"/>
+  <xacro:include filename="$(find benzene_description)/urdf/sensors/ultrasonic_sensor.xacro"/>
+  <xacro:include filename="$(find benzene_description)/urdf/mech/caster.xacro"/>
+  <xacro:include filename="$(find benzene_description)/urdf/mech/wheel.xacro"/>
+  <xacro:include filename="$(find benzene_description)/urdf/mech/base.xacro"/>
+  <xacro:base
+    prefix="$(arg prefix)"
+    base_name="base"
+    parent="base_footprint"
+    xyz_offset="0 0 0"
+    rpy_offset="0 0 0"
+    base_length="${base_length}"
+    base_width="${base_width}"
+    base_height="${base_height}"
+    base_mass="${base_mass}"/>
   <xacro:lidar_sensor
     prefix="$(arg prefix)"
@@ -239,24 +58,52 @@
     topic="camera/image_raw"
     camera_info_topic="camera/camera_info"/>
-  <joint name="uss_joint" type="fixed">
-    <parent link="base_link"/>
-    <child link="uss_link"/>
-    <origin xyz="0.175 0 0.055" rpy="0 0 0"/>
-  </joint>
-  <link name="uss_link"/>
+  <xacro:caster_wheel
+    prefix="$(arg prefix)"
+    caster_name="front_caster_wheel"
+    parent="base_link"
+    xyz_offset="0.13 0 0"
+    rpy_offset="0 0 0"
+    caster_radius="${caster_radius}"
+    caster_mass="${caster_mass}"/>
+  <xacro:caster_wheel
+    prefix="$(arg prefix)"
+    caster_name="back_caster_wheel"
+    parent="base_link"
+    xyz_offset="-0.13 0 0"
+    rpy_offset="0 0 0"
+    caster_radius="${caster_radius}"
+    caster_mass="${caster_mass}"/>
+  <xacro:wheel
+    prefix="$(arg prefix)"
+    wheel_name="left_wheel"
+    parent="base_link"
+    xyz_offset="0 0.0925 0.020"
+    rpy_offset="0 0 0"
+    axis="0 1 0"
+    wheel_radius="${wheel_radius}"
+    wheel_width="${wheel_width}"
+    wheel_mass="${wheel_mass}"/>
+  <xacro:wheel
+    prefix="$(arg prefix)"
+    wheel_name="right_wheel"
+    parent="base_link"
+    xyz_offset="0 -0.0925 0.020"
+    rpy_offset="0 0 0"
+    axis="0 1 0"
+    wheel_radius="${wheel_radius}"
+    wheel_width="${wheel_width}"
+    wheel_mass="${wheel_mass}"/>
+  <xacro:ultrasonic_sensor
+    prefix="$(arg prefix)"
+    sensor_name="ultrasonic_link"
+    parent="base_link"
+    xyz_offset="0.175 0 0.055"
+    rpy_offset="0 0 0"
+    topic_name="ultrasonic_link/data"/>
   <xacro:include filename="$(find benzene_description)/urdf/control/gazebo_sim_ros2_control.urdf.xacro"/>
-  <xacro:load_gazebo_sim_ros2_control_plugin robot_name="benzene" use_gazebo="$(arg use_gazebo)"/>
+  <xacro:load_gazebo_sim_ros2_control_plugin robot_name="$(arg robot_name)" use_gazebo="$(arg use_gazebo)"/>
   <xacro:include filename="$(find benzene_description)/urdf/control/velocity_control_plugin.urdf.xacro"/>
   <xacro:load_velocity_control_plugin use_gazebo="$(arg use_gazebo)"/>
   <xacro:include filename="$(find benzene_description)/urdf/control/benzene_control.urdf.xacro"/>
   <xacro:benzene_ros2_control prefix="$(arg prefix)" use_gazebo="$(arg use_gazebo)"/>
-  <gazebo reference="$(arg prefix)back_caster_wheel">
-    <material>
-      <ambient>0 0 0 1</ambient>
-      <diffuse>0 0 0 1</diffuse>
-      <specular>0 0 0 1</specular>
-    </material>
-    <mu1>0.0001</mu1>
-    <mu2>0.0001</mu2>
-  </gazebo>
 </robot>

File: benzene_description/urdf/sensors/simple_camera.xacro (robot description, xacro)
@@ -24,13 +24,9 @@
     camera_info_topic:='camera/camera_info'
   ">
-    <!-- Camera Body -->
     <link name="${prefix}${camera_name}_link">
       <visual>
-        <origin
-          xyz="0 0 0"
-          rpy="0 0 0"/>
+        <origin xyz="0 0 0" rpy="0 0 0"/>
         <geometry>
-          <box
-            size="${cam_depth} ${cam_width} ${cam_height}"/>
+          <box size="${cam_depth} ${cam_width} ${cam_height}"/>
         </geometry>
         <material name="${material_name}">
@@ -39,31 +35,18 @@
       </visual>
     </link>
-    <!-- Camera Mount Joint -->
-    <joint
-      name="${prefix}${camera_name}_joint"
-      type="fixed">
+    <joint name="${prefix}${camera_name}_joint" type="fixed">
       <parent link="${prefix}${parent}"/>
       <child link="${prefix}${camera_name}_link"/>
-      <origin
-        xyz="${xyz_offset}"
-        rpy="${rpy_offset}"/>
+      <origin xyz="${xyz_offset}" rpy="${rpy_offset}"/>
     </joint>
-    <!-- Optical Frame -->
     <link name="${prefix}${camera_name}_optical"/>
-    <joint
-      name="${prefix}${camera_name}_optical_joint"
-      type="fixed">
+    <joint name="${prefix}${camera_name}_optical_joint" type="fixed">
       <parent link="${prefix}${camera_name}_link"/>
       <child link="${prefix}${camera_name}_optical"/>
-      <origin
-        xyz="0 0 0"
-        rpy="${-M_PI/2} 0 ${-M_PI/2}"/>
+      <origin xyz="0 0 0" rpy="0 0 0"/>
     </joint>
-    <!-- Gazebo Simple RGB Camera -->
     <gazebo reference="${prefix}${camera_name}_link">
       <material>Gazebo/Black</material>
-      <sensor
-        name="${prefix}${camera_name}"
-        type="camera">
+      <sensor name="${prefix}${camera_name}" type="camera">
         <pose>0 0 0 0 0 0</pose>
         <always_on>${always_on}</always_on>
