Commit message: added switch between worlds for gazebo.sh too, made cleaner .sh files, removed all depth cam related code from nav urdf cam gz bridge nav rviz. adjusted april tag in cafe world

File: benzene_description/urdf/robots/benzene.urdf.xacro (robot description, xacro)
@@ -48,5 +48,5 @@
     topic_name="imu/data"/>
   <xacro:simple_camera
-    camera_name="camera"
+    camera_name="cam_1"
     parent="base_link"
     xyz_offset="0.17 0 0.03"
@@ -56,6 +56,6 @@
     horizontal_fov="1.089"
     update_rate="30"
-    topic="camera/image_raw"
-    camera_info_topic="camera/camera_info"/>
+    topic="cam_1/image_raw"
+    camera_info_topic="cam_1/camera_info"/>
   <xacro:caster_wheel
     prefix="$(arg prefix)"

File: benzene_description/urdf/sensors/simple_camera.xacro (robot description, xacro)
@@ -44,5 +44,5 @@
       <parent link="${prefix}${camera_name}_link"/>
       <child link="${prefix}${camera_name}_optical"/>
-      <origin xyz="0 0 0" rpy="0 0 0"/>
+      <origin xyz="0 0 0" rpy="${-M_PI/2} 0 ${-M_PI/2}"/>
     </joint>
     <gazebo reference="${prefix}${camera_name}_link">

Commit message: Added and updated ultrasonic in the gazebo, yet to add in the navigation code

File: benzene_description/urdf/robots/benzene.urdf.xacro (robot description, xacro)
@@ -96,9 +96,9 @@
   <xacro:ultrasonic_sensor
     prefix="$(arg prefix)"
-    sensor_name="ultrasonic_link"
+    sensor_name="ultrasonic"
     parent="base_link"
     xyz_offset="0.175 0 0.055"
     rpy_offset="0 0 0"
-    topic_name="ultrasonic_link/data"/>
+    topic_name="ultrasonic/scan"/>
   <xacro:include filename="$(find benzene_description)/urdf/control/gazebo_sim_ros2_control.urdf.xacro"/>
   <xacro:load_gazebo_sim_ros2_control_plugin robot_name="$(arg robot_name)" use_gazebo="$(arg use_gazebo)"/>

File: benzene_description/urdf/sensors/ultrasonic_sensor.xacro (robot description, xacro)
@@ -1,5 +1,5 @@
 <?xml version="1.0"?>
 <robot xmlns:xacro="http://www.ros.org/wiki/xacro">
-  <xacro:macro name="ultrasonic_sensor" params="
+<xacro:macro name="ultrasonic_sensor" params="
     prefix:=''
     sensor_name:='ultrasonic'
@@ -11,39 +11,54 @@
     material_name:='black'
     material_color:='0 0 0 1'
-    topic_name:='ultrasonic/data'
+    topic_name:='ultrasonic/scan'
+    update_rate:=10
+    min_range:=0.02
+    max_range:=4.0
   ">
-    <link name="${prefix}${sensor_name}">
-      <visual>
-        <origin xyz="0 0 0" rpy="0 0 0"/>
-      </visual>
-    </link>
-    <joint name="${prefix}${sensor_name}_joint" type="fixed">
-      <parent link="${prefix}${parent}"/>
-      <child link="${prefix}${sensor_name}"/>
-      <origin xyz="${xyz_offset}" rpy="${rpy_offset}"/>
-    </joint>
-    <gazebo reference="${prefix}${sensor_name}">
-      <sensor name="${prefix}${sensor_name}" type="ray">
-        <pose> 0 0 0 0 0 0 </pose>
-        <visualize>true</visualize>
-        <update_rate>10</update_rate>
-        <ray>
-          <scan>
-            <horizontal>
-              <samples>1</samples>
-              <resolution>1</resolution>
-              <min_angle>0</min_angle>
-              <max_angle>0</max_angle>
-            </horizontal>
-          </scan>
-          <range>
-            <min>0.02</min>
-            <max>4.0</max>
-            <resolution>0.01</resolution>
-          </range>
-        </ray>
-        <topic>${topic_name}</topic>
-      </sensor>
-    </gazebo>
-  </xacro:macro>
+  <link name="${prefix}${sensor_name}">
+    <visual>
+      <origin xyz="0 0 0" rpy="0 ${pi/2} 0"/>
+      <geometry>
+        <cylinder radius="${sensor_radius}" length="${sensor_length}"/>
+      </geometry>
+      <material name="${material_name}">
+        <color rgba="${material_color}"/>
+      </material>
+    </visual>
+  </link>
+  <joint name="${prefix}${sensor_name}_joint" type="fixed">
+    <parent link="${prefix}${parent}"/>
+    <child link="${prefix}${sensor_name}"/>
+    <origin xyz="${xyz_offset}" rpy="${rpy_offset}"/>
+  </joint>
+  <gazebo reference="${prefix}${sensor_name}">
+    <sensor name="${prefix}${sensor_name}" type="gpu_lidar">
+      <always_on>true</always_on>
+      <visualize>true</visualize>
+      <update_rate>${update_rate}</update_rate>
+      <topic>${topic_name}</topic>
+      <gz_frame_id>${prefix}${sensor_name}</gz_frame_id>
+      <lidar>
+        <scan>
+          <horizontal>
+            <samples>5</samples>
+            <resolution>1</resolution>
+            <min_angle>-0.13</min_angle>
+            <max_angle>0.13</max_angle>
+          </horizontal>
+        </scan>
+        <range>
+          <min>${min_range}</min>
+          <max>${max_range}</max>
+          <resolution>0.01</resolution>
+        </range>
+        <noise>
+          <type>gaussian</type>
+          <mean>0.0</mean>
+          <stddev>0.01</stddev>
+        </noise>
+      </lidar>
+    </sensor>
+  </gazebo>
+</xacro:macro>
 </robot>
